File: PCB/rc.kicad_sch (KiCad schematic)
At the start: 5 parts, among them J1 USB_C_Receptacle_USB2.0_16P, J2 USB_A, J3 Conn_01x07_Pin, U1 ESP32-S3-WROOM-1U, U2 MAX3421EEHJ+T

Commit message: pcb init
Parts:
- added C1, C2: C, Capacitor_SMD:C_0402_1005Metric_Pad0.74x0.62mm_HandSolder, symbol Device:C
- added U3: ME6211C33M5, Package_TO_SOT_SMD:SOT-23-5, symbol Regulator_Linear:ME6211C33M5
- J3: value Conn_01x07_Pin -> OLED display
Connections:
- net at J1.A1 (GND), J1.A12 (GND), J1.B1 (GND)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: now also J3.1 (Pin_1), U2.19 (GND), U2.3 (GND), C1.2, C2.2, U3.2 (V_{SS})
- net at J1.A4 (VBUS), J1.A9 (VBUS), J1.B4 (VBUS)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: now also C1.1, U3.1 (V_{IN}), U3.3 (CE)
- net at J1.A6 (D+): now also J1.B6 (D+), U1.14 (IO20)
- net at J1.A7 (D-): now also J1.B7 (D-), U1.13 (IO19)
- net at U1.18 (IO10): now also U2.14 (*SS)
- net at U1.19 (IO11): now also J3.4 (Pin_4), U2.16 (MOSI)
- net at U1.2 (3V3): now also J3.2 (Pin_2), U2.23 (VCC), C2.1, U3.5 (V_{OUT})
- net at U1.20 (IO12): now also J3.3 (Pin_3), U2.13 (SCLK)
- net at U1.21 (IO13): now also U2.15 (MISO)
- net at U1.22 (IO14): now also J3.5 (Pin_5)
- net at U1.8 (IO15): now also J3.6 (Pin_6)
- net at U1.9 (IO16): now also J3.7 (Pin_7)
Other:
- moved on the sheet: J3, U2

Commit message: pcb update
Parts:
- added C3, C4, C5, C7: C, Capacitor_SMD:C_0402_1005Metric_Pad0.74x0.62mm_HandSolder, symbol Device:C
- added D1, D2: ESD9B5.0ST5G, Diode_SMD:D_SOD-923, symbol Diode:ESD9B5.0ST5G
- added FB1, FB2: FerriteBead, Inductor_SMD:L_0603_1608Metric, symbol Device:FerriteBead
- added R1, R2, R3: R_US, Resistor_SMD:R_0402_1005Metric_Pad0.72x0.64mm_HandSolder, symbol Device:R_US
- added Y1: Crystal, Crystal:Crystal_SMD_G8-2Pin_3.2x1.5mm, symbol Device:Crystal
- J3: footprint Connector_PinSocket_1.27mm:PinSocket_1x07_P1.27mm_Vertical -> Connector_PinSocket_2.54mm:PinSocket_1x07_P2.54mm_Horizontal
Connections:
- net at C1.1, J1.A4 (VBUS), J1.A9 (VBUS)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: now also FB2.2; no longer J2.1 (VBUS)
- net at C1.2, C2.2, J1.A1 (GND)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: now also C3.1, C4.1, C5.2, C7.2, FB1.2
- net at U1.17 (IO9): now also U2.18 (INT), R3.1
- net at C2.1, J3.2 (Pin_2), U1.2 (3V3)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: now also U1.3 (EN), U2.2 (VL), R3.2
- net at J2.2 (D-): now also R1.1
- net at J2.3 (D+): now also R2.1
- net at U2.20 (D-): now also D2.1 (A1), R1.2
- net at U2.21 (D+): now also D1.1 (A1), R2.2
- net at U2.22 (VBCOMP): now also C7.1
- net at U2.24 (XI): now also C4.2, Y1.1
- net at U2.25 (XO): now also C3.2, Y1.2
- new net: D1.2 (A2), D2.2 (A2), FB1.1
- new net: C5.1, FB2.1, J2.1 (VBUS)

Commit message: 3 inch display
Parts:
- removed J3: OLED display, Connector_PinSocket_2.54mm:PinSocket_1x07_P2.54mm_Horizontal, symbol Connector:Conn_01x07_Pin
- added J3: Conn_02x08_Odd_Even, Connector_PinSocket_2.54mm:PinSocket_2x08_P2.54mm_Vertical, symbol Connector_Generic:Conn_02x08_Odd_Even
- added SW1, SW2, SW3: SW_Omron_B3FS, Button_Switch_SMD:SW_SPST_Omron_B3FS-105xP, symbol Switch:SW_Omron_B3FS
- J1: footprint Connector_USB:USB_C_Receptacle_GCT_USB4110 -> usbc:GCT_USB4120-03-C_REVA
- J2: footprint Connector_USB:USB_A_Molex_67643_Horizontal -> usb-a vertical:ONSHORE_USB-A1VSB6
Connections:
- net CS: now also U1.9 (IO16), J3.16 (Pin_16)
- net DC: now also U1.8 (IO15), J3.14 (Pin_14)
- net GND: now also C1.2, C2.2, C3.1, C4.1, C5.2, C7.2, FB1.2, J1.A1 (GND), J1.A12 (GND), J1.B1 (GND), J1.B12 (GND), J1.S1 (SHIELD), J2.4 (GND), J2.5 (Shield), U1.1 (GND), U1.40 (GND), U1.41 (GND), U2.19 (GND), U2.3 (GND), U3.2 (V_{SS}), J3.1 (Pin_1), SW1.1, SW2.1, SW3.1
- net RES: now also U1.22 (IO14), J3.15 (Pin_15)
- net at C2.1, R3.2, U1.2 (3V3)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: now also J3.2 (Pin_2)
- net MOSI: now reaches U1.19 (IO11), U2.16 (MOSI)
- net MOSI: now also J3.5 (Pin_5)
- net CLK: now reaches U1.20 (IO12), U2.13 (SCLK)
- net CLK: now also J3.4 (Pin_4)
- net at U1.23 (IO21): now also SW3.2
- net at U1.35 (IO42): now also SW1.2
- net at U1.7 (IO7): now also SW2.2
Other:
- moved on the sheet: C1, C2, C3, C4, C5, C7, D1, D2, FB1, FB2, J1, J2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

Commit message: more board
Parts:
- removed D1, D2: ESD9B5.0ST5G, Diode_SMD:D_SOD-923, symbol Diode:ESD9B5.0ST5G
- added C6: 100nf, Capacitor_SMD:C_0402_1005Metric_Pad0.74x0.62mm_HandSolder, symbol Device:C
- added D3, D4: PGB1010603MR, esd:DIOC1608X36N, symbol esd:PGB1010603MR
- added R4, R5: 5.1k, Resistor_SMD:R_0402_1005Metric_Pad0.72x0.64mm_HandSolder, symbol Device:R_US
- C1, C2: value C -> 10mfd
- C3, C4: value C -> 22pf
- C7: value C -> 0.1mfd
- R1, R2: value R_US -> 22
- R3: value R_US -> 10k
- Y1: value Crystal -> 12Mhz/12pf
Connections:
- net GND: now also C6.2, R4.2, R5.2
- net at J1.A5 (CC1): now also R4.1
- net at J1.B5 (CC2): now also R5.1
- net at R1.2, U2.20 (D-): now also D4.1
- net at FB1.1: now also D3.2, D4.2
- net at C2.1, J3.2 (Pin_2), R3.2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: now also C6.1
- net at R2.2, U2.21 (D+): now also D3.1
Other:
- moved on the sheet: C2
